File: hw/rev0/vehicle_control_module.brd (EAGLE design)
At the start: 160 x 100 mm, 286 parts, among them IC1 SJA1105TELY, IC10 TJA1100HNZ, IC11 KSZ8061MNXI-TR, IC12 TJA1100HNZ, IC14 NUP2202W1T2G, IC15 TLE9252VSKXUMA1, IC16 NUP2202W1T2G, IC17 LP5907QMFX-3.3Q1, IC2 ATSAMV71Q21B-AABT, IC3 TJA1100HNZ, IC4 FT2232HL, IC5 TRS3232EQPWRQ1, IC6 SST26VF032BT-104I_SM, IC7 DS3231SN#, IC8 TLE9252VSKXUMA1, IC9 TPS62242DRVR, J10 5-2337992-3, J11 2301843-1, J12 1017505, J13 2301843-1, J15 693022010811, J2 2305018-2, J27 2041119-2, J3 1017505, J4 1017505, J5 1017505, J6 1017505, J7 1017505, J8 1017505, J9 1017505, U1 122-2920-GR, U2 LM63625, U3 TPS62007-Q1_DGS_10, Y1 NX3225SA-25MHZ-EXS00A-CS11338, Y2 NX2016SA-25.000M-STD-CZS-1, Y3 ABM8AIG-12.000MHZ-1Z-T

Commit message: Add high side drivers
Parts:
- added C108, C111, C114, C116, C118, C120, C122, C124, C126, C128, C130, C132, C134, C136, C138, C140, C142, C144: 0.01uF, rcl:C0603
- added C112, C113, C115, C117, C119, C121, C123, C125, C127, C129, C131, C133, C135, C137, C139, C141, C143, C145: 150nF, rcl:C0603
- added D10, D11, D12, D13, D14, D15, D16, D17, D18, D19, D20, D21, D22, D23, D24, D25, D26, D27: BAT54SWFILMY, samacsys:SOT65P210X110-3N
- added LED10, LED11, LED12, LED8: (no value), led:CHIPLED_0603
- added R100, R101, R103, R104: 10k, rcl:R0603
- added R105, R106, R115, R120, R125, R130, R135, R140, R145, R150, R155, R160, R165, R170, R175, R180, R185, R190: 4, rcl:R1206
- added R107, R110, R111, R114, R116, R119, R121, R124, R126, R129, R131, R134, R136, R139, R141, R144, R146, R149, R151, R154, R156, R159, R161, R164, R166, R169, R171, R174, R176, R179, R181, R184, R186, R189, R191, R194: 4.7k, rcl:R0603
- added R108, R112, R117, R122, R127, R132, R137, R142, R147, R152, R157, R162, R167, R172, R177, R182, R187, R192: 2.74k, rcl:R0603
- added R109, R113, R118, R123, R128, R133, R138, R143, R148, R153, R158, R163, R168, R173, R178, R183, R188, R193: 1k, rcl:R0603
- added U?10, U?11, U?12, U?13, U?14, U?15, U?16, U?17, U?18, U?2, U?3, U?4, U?5, U?6, U?7, U?8, U?9: (no value), BTS50015-1TAD:TO127P1500X450-7_8N-V1
Connections:
- removed net VS: U?1.8
- new net HIGHSIDE_0_EN: R154.2
- new net HIGHSIDE_0_OUTPUT: U?10.5, U?10.6, U?10.7
- new net HIGHSIDE_10_EN: R114.2
- new net HIGHSIDE_10_OUTPUT: U?2.5, U?2.6, U?2.7
- new net HIGHSIDE_11_EN: R119.2
- new net HIGHSIDE_11_OUTPUT: U?3.5, U?3.6, U?3.7
- new net HIGHSIDE_12_EN: R124.2
- new net HIGHSIDE_12_OUTPUT: U?4.5, U?4.6, U?4.7
- new net HIGHSIDE_13_EN: R129.2
- new net HIGHSIDE_13_OUTPUT: U?5.5, U?5.6, U?5.7
- new net HIGHSIDE_14_EN: R134.2
- new net HIGHSIDE_14_OUTPUT: U?6.5, U?6.6, U?6.7
- new net HIGHSIDE_15_EN: R139.2
- new net HIGHSIDE_15_OUTPUT: U?7.5, U?7.6, U?7.7
- new net HIGHSIDE_16_EN: R144.2
- new net HIGHSIDE_16_OUTPUT: U?8.5, U?8.6, U?8.7
- new net HIGHSIDE_17_EN: R149.2
- new net HIGHSIDE_17_OUTPUT: U?9.5, U?9.6, U?9.7
- new net HIGHSIDE_1_EN: R159.2
- new net HIGHSIDE_1_OUTPUT: U?11.5, U?11.6, U?11.7
- new net HIGHSIDE_2_EN: R164.2
- new net HIGHSIDE_2_OUTPUT: U?12.5, U?12.6, U?12.7
- new net HIGHSIDE_3_EN: R169.2
- new net HIGHSIDE_3_OUTPUT: U?13.5, U?13.6, U?13.7
- new net HIGHSIDE_4_EN: R174.2
- new net HIGHSIDE_4_OUTPUT: U?14.5, U?14.6, U?14.7
- new net HIGHSIDE_5_EN: R179.2
- new net HIGHSIDE_5_OUTPUT: U?15.5, U?15.6, U?15.7
- new net HIGHSIDE_6_EN: R184.2
- new net HIGHSIDE_6_OUTPUT: U?16.5, U?16.6, U?16.7
- new net HIGHSIDE_7_EN: R189.2
- new net HIGHSIDE_7_OUTPUT: U?17.5, U?17.6, U?17.7
- new net HIGHSIDE_8_EN: R194.2
- new net HIGHSIDE_8_OUTPUT: U?18.5, U?18.6, U?18.7
- new net HIGHSIDE_9_EN: R110.2
- new net HIGHSIDE_9_OUTPUT: U?1.5, U?1.6, U?1.7
- new net N$100: R115.1, U?3.1
- new net N$101: R116.1, R117.1, U?3.3
- new net N$102: C115.1, R118.1, R119.1, U?3.2
- new net N$103: R120.1, U?4.1
- new net N$104: R121.1, R122.1, U?4.3
- new net N$105: C117.1, R123.1, R124.1, U?4.2
- new net N$106: R125.1, U?5.1
- new net N$107: R126.1, R127.1, U?5.3
- new net N$108: C119.1, R128.1, R129.1, U?5.2
- new net N$109: R130.1, U?6.1
- new net N$110: R131.1, R132.1, U?6.3
- new net N$111: C121.1, R133.1, R134.1, U?6.2
- new net N$112: R135.1, U?7.1
- new net N$113: R136.1, R137.1, U?7.3
- new net N$114: C123.1, R138.1, R139.1, U?7.2
- new net N$115: R140.1, U?8.1
- new net N$116: R141.1, R142.1, U?8.3
- new net N$117: C125.1, R143.1, R144.1, U?8.2
- new net N$118: R145.1, U?9.1
- new net N$119: R146.1, R147.1, U?9.3
- new net N$120: C127.1, R148.1, R149.1, U?9.2
- new net N$121: R150.1, U?10.1
- new net N$122: R151.1, R152.1, U?10.3
- new net N$123: C129.1, R153.1, R154.1, U?10.2
- new net N$124: R155.1, U?11.1
- new net N$125: R156.1, R157.1, U?11.3
- new net N$126: C131.1, R158.1, R159.1, U?11.2
- new net N$127: R160.1, U?12.1
- new net N$128: R161.1, R162.1, U?12.3
- new net N$129: C133.1, R163.1, R164.1, U?12.2
- new net N$130: R165.1, U?13.1
- new net N$131: R166.1, R167.1, U?13.3
- new net N$132: C135.1, R168.1, R169.1, U?13.2
- new net N$133: R170.1, U?14.1
- new net N$134: R171.1, R172.1, U?14.3
- new net N$135: C137.1, R173.1, R174.1, U?14.2
- new net N$136: R175.1, U?15.1
- new net N$137: R176.1, R177.1, U?15.3
- new net N$138: C139.1, R178.1, R179.1, U?15.2
- new net N$139: R180.1, U?16.1
- new net N$140: R181.1, R182.1, U?16.3
- new net N$141: C141.1, R183.1, R184.1, U?16.2
- new net N$142: R185.1, U?17.1
- new net N$143: R186.1, R187.1, U?17.3
- new net N$144: C143.1, R188.1, R189.1, U?17.2
- new net N$145: R190.1, U?18.1
- new net N$146: R191.1, R192.1, U?18.3
- new net N$147: C145.1, R193.1, R194.1, U?18.2
- new net N$88: LED8.A, R100.2
- new net N$90: LED10.A, R101.2
- new net N$91: LED11.A, R103.2
- new net N$93: LED12.A, R104.2
- new net N$94: R106.1, U?1.1
- new net N$95: R107.1, R108.1, U?1.3
- new net N$96: R105.1, U?2.1
- new net N$97: C112.1, R109.1, R110.1, U?1.2
- new net N$98: R111.1, R112.1, U?2.3
- new net N$99: C113.1, R113.1, R114.1, U?2.2
- net +3V3: now also D10.2, D11.2, D12.2, D13.2, D14.2, D15.2, D16.2, D17.2, D18.2, D19.2, D20.2, D21.2, D22.2, D23.2, D24.2, D25.2, D26.2, D27.2, R103.1
- net +5V: now also R104.1
- net 3V3_AD_REF: now also R100.1
- net ADC0_10: now also C140.1, D25.3, R181.2
- net ADC0_3: now also C128.1, D19.3, R151.2
- net ADC0_4: now also C130.1, D20.3, R156.2
- net ADC0_6: now also C132.1, D21.3, R161.2
- net ADC0_7: now also C134.1, D22.3, R166.2
- net ADC0_8: now also C136.1, D23.3, R171.2
- net ADC0_9: now also C138.1, D24.3, R176.2
- net ADC1_0: now also C142.1, D26.3, R186.2
- net ADC1_1: now also C144.1, D27.3, R191.2
- net ADC1_10: now also C124.1, D17.3, R141.2
- net ADC1_11: now also C126.1, D18.3, R146.2
- net ADC1_2: now also C111.1, D10.3, R107.2
- net ADC1_4: now also C108.1, D11.3, R111.2
- net ADC1_5: now also C114.1, D12.3, R116.2
- net ADC1_6: now also C116.1, D13.3, R121.2
- net ADC1_7: now also C118.1, D14.3, R126.2
- net ADC1_8: now also C120.1, D15.3, R131.2
- net ADC1_9: now also C122.1, D16.3, R136.2
- net GND: now also C108.2, C111.2, C112.2, C113.2, C114.2, C115.2, C116.2, C117.2, C118.2, C119.2, C120.2, C121.2, C122.2, C123.2, C124.2, C125.2, C126.2, C127.2, C128.2, C129.2, C130.2, C131.2, C132.2, C133.2, C134.2, C135.2, C136.2, C137.2, C138.2, C139.2, C140.2, C141.2, C142.2, C143.2, C144.2, C145.2, D10.1, D11.1, D12.1, D13.1, D14.1, D15.1, D16.1, D17.1, D18.1, D19.1, D20.1, D21.1, D22.1, D23.1, D24.1, D25.1, D26.1, D27.1, LED10.C, LED11.C, LED12.C, LED8.C, R105.2, R106.2, R108.2, R109.2, R112.2, R113.2, R115.2, R117.2, R118.2, R120.2, R122.2, R123.2, R125.2, R127.2, R128.2, R130.2, R132.2, R133.2, R135.2, R137.2, R138.2, R140.2, R142.2, R143.2, R145.2, R147.2, R148.2, R150.2, R152.2, R153.2, R155.2, R157.2, R158.2, R160.2, R162.2, R163.2, R165.2, R167.2, R168.2, R170.2, R172.2, R173.2, R175.2, R177.2, R178.2, R180.2, R182.2, R183.2, R185.2, R187.2, R188.2, R190.2, R192.2, R193.2; no longer U?1.1
- net VBATT: now also U?1.8, U?10.8, U?11.8, U?12.8, U?13.8, U?14.8, U?15.8, U?16.8, U?17.8, U?18.8, U?2.8, U?3.8, U?4.8, U?5.8, U?6.8, U?7.8, U?8.8, U?9.8
- net VDD: now also R101.1
