File: hw/rev0/vehicle_control_module.sch (EAGLE design)
At the start: 247 parts, among them IC1 SJA1105TELY, IC10 TJA1100HNZ, IC11 KSZ8061MNXI-TR, IC12 TJA1100HNZ, IC13 TPS79133MDBVTEP, IC2 ATSAMV71Q21B-AABT, IC3 TJA1100HNZ, IC4 FT2232HL, IC5 TRS3232EQPWRQ1, IC6 SST26VF032BT-104I_SM, IC7 DS3231SN#, IC8 TLE9252VSKXUMA1, IC9 TPS62242DRVR, J1 2305018-2, J10 5-2337992-3, J11 2301843-1, J12 1017505, J13 2301843-1, J2 2305018-2, J3 1017505, J4 1017505, J5 1017505, J6 1017505, J7 1017505, J8 1017505, J9 1017505, U1 122-2920-GR, U2 LM63625, U3 TPS62007-Q1_DGS_10, Y1 NX3225SA-25MHZ-EXS00A-CS11338, Y2 NX2016SA-25.000M-STD-CZS-1, Y3 ABM8AIG-12.000MHZ-1Z-T

Commit message: Add LTE modem and flesh out CAN interface
Parts:
- removed J1: 2305018-2, 2305018-2:2305018-2
- added C89: 0.1uF, rcl:C-USC0603
- added C90, C93: 4.7nF, rcl:C-USC0603
- added C91, C92, C94, C95, C98: 100nF, rcl:C-USC0603
- added C96: 1uF, rcl:C-USC0603
- added C97: UCZ1K151MNQ1MS, samacsys:UCZ1K151MNQ1MS
- added IC14, IC16: NUP2202W1T2G, samacsys:NUP2202W1T2G
- added IC15: TLE9252VSKXUMA1, samacsys:TLE9252VSKXUMA1
- added J15: 693022010811, samacsys:693022010811
- added J27: 2041119-2, samacsys:2041119-2
- added LED9: (no value), led:LEDCHIPLED_0603
- added R102: 10k, rcl:R-US_R0603
- added R94: 1.21k, rcl:R-US_R0603
- added R95, R96: 60, rcl:R-US_R0805
- R1, R2: value 5.11k -> 60; device rcl:R-US_R0603 -> rcl:R-US_R0805
Connections:
- removed net HOST_USB_VBUS: J1.VBUS_A, J1.VBUS_B
- removed net N$2: J1.CC1, R1.2
- removed net N$43: IC11.VDDIO
- new net CAN0_EN: IC2.PA22, IC8.EN
- new net CAN0_ERR: IC2.PC2, IC8.NERR
- new net CAN0_H: IC14.I/O_1, IC8.CANH, R1.1
- new net CAN0_INH: IC8.INH
- new net CAN0_L: IC14.I/O_2, IC8.CANL, R2.2
- new net CAN0_STBY: IC2.PC1, IC8.NSTB
- new net CAN1_EN: IC15.EN, IC2.PC11
- new net CAN1_ERR: IC15.NERR, IC2.PC10
- new net CAN1_H: IC15.CANH, IC16.I/O_1, R95.1
- new net CAN1_INH: IC15.INH
- new net CAN1_L: IC15.CANL, IC16.I/O_2, R96.2
- new net CAN1_STBY: IC15.NSTB, IC2.PA2
- new net MODEM_DISABLE: IC2.PB9, J27.W_DISABLE#
- new net MODEM_RESET: IC2.PB8, J27.PERST#
- new net MODEM_WAN_LED: J27.LED_WWAN#, LED9.C
- new net N$92: LED9.A, R102.2
- new net RTC_RESET: IC2.PD13, IC7.!RST
- new net SIM_CLK: J15.CLK, J27.UIM_CLK
- new net SIM_DATA: J15.I/O, J27.UIM_DATA
- new net SIM_PWR: J15.VCC, J15.VPP, J27.UIM_PWR
- new net SIM_RESET: J15.RST, J27.UIM_RESET
- new net VBATT_PROT: C86.+, C87.1, C88.1, IC15.VBAT, IC15.WAKE, IC8.VBAT, IC8.WAKE, L7.2, R93.1, U2.VIN, U2.VIN_2
- net +3V3: now also C91.1, C92.1, C94.1, C95.1, C96.1, C97.+, C98.1, IC11.VDDIO, IC14.VP, IC15.VCC, IC15.VIO, IC16.VP, IC8.VCC, IC8.VIO, J27.+3.3VAUX_1, J27.+3.3VAUX_2, J27.+3.3VAUX_3, J27.+3.3VAUX_4, J27.3.3VAUX, R102.1
- net ADC0_0: now also C89.1, R93.2, R94.2
- net CAN0_RX: now also IC8.RXD
- net CAN0_TX: now also IC8.TXD
- net CAN1_RX: now also IC15.RXD
- net CAN1_TX: now also IC15.TXD
- net GND: now also C89.2, C90.2, C91.2, C92.2, C93.2, C94.2, C95.2, C96.2, C97.-, C98.2, IC14.VN, IC15.GND, IC16.VN, IC2.GND_1, IC2.GND_2, IC2.GND_3, IC2.GND_4, IC2.GND_5, IC2.GND_6, IC8.GND, J15.GND, J27.GND_1, J27.GND_10, J27.GND_11, J27.GND_12, J27.GND_13, J27.GND_14, J27.GND_2, J27.GND_3, J27.GND_4, J27.GND_5, J27.GND_6, J27.GND_7, J27.GND_8, J27.GND_9, J27.RESERVED_1, R94.1; no longer J1.GND, J1.GNDA, J1.GNDB, J1.SHIELD, R1.1, R2.1
- net HOST_USB_DM: now also J27.USB_D-; no longer J1.DA_N, J1.DB_N
- net HOST_USB_DP: now also J27.USB_D+; no longer J1.DA_P, J1.DB_P
- net N$3: now also C93.1, R95.2, R96.1; no longer J1.CC2, R2.2
- net N$82: now also C90.1, R1.2, R2.1; no longer C86.+, C87.1, C88.1, L7.2, U2.VIN, U2.VIN_2
Other:
- note added: "10. High-side drivers"
- note added: "12. Modem"
- note added: "13. Connectors"
- note added: "3. RS232 and debug UART"
- note added: "9. Ethernet PHY 4 (100BASE-TX)"
- note added: "Breakdown Voltage = 29.5V"
- note added: "MicroSIM socket"
- note added: "RC cutoff ~160Hz"
- note removed: "12. Connectors"

Commit message: First stab at power supply
Parts:
- added C100, C99: 470pF, rcl:C-USC0805
- added C101: 0.47uF, rcl:C-USC0603
- added C102: 220nF, rcl:C-USC0805
- added C103, C104, C105, C107: 10uF, rcl:C-USC0805
- added C106, C109: 1uF, rcl:C-USC0603
- added C108: 0.01uF, rcl:C-USC0603
- added C110: 0.1uF, rcl:C-USC0603
- added D6, D9: PMEG3030EP,115, samacsys:PMEG3030EP,115
- added D8: SMAJ24CA-Q, samacsys:SMAJ24CA-Q
- added L10: LPS3015-222MRB, samacsys:LPS3015-222MRB
- added L8: XAL4040-103MEC, samacsys:XAL4040-103MEC
- added L9: DO3316P-103MLB, samacsys:DO3316P-103MLB
- added R100, R101: 1k, rcl:R-US_R0603
- added R97: 1k, rcl:R-US_R0805
- added R98: 10k, rcl:R-US_R0603
- added R99: 0, rcl:R-US_R0603
- C84, C85: device rcl:C-USC0603 -> rcl:C-USC0805
Connections:
- removed net CAN0_INH: IC8.INH
- removed net CAN1_INH: IC15.INH
- new net +5V: C103.1, C107.1, C110.1, IC13.IN, IC9.VIN, L8.2, U2.FB, U3.ILIM, U3.VIN
- new net 1V2_SUPPLY_EN: IC9.EN, R100.2
- new net 3V3_AD_REF: C109.1, IC13.OUT
- new net 3V3_AD_SUPPLY_EN: IC13.!EN, R101.2
- new net MAIN_SUPPLY_PGOOD: R98.1, U2.RESET_N, U3.EN
- new net N$2: C100.1, C99.2
- new net N$43: D6.K, D9.K, R97.2, U2.EN
- new net N$83: C101.1, R98.2, U2.RT, U2.VCC, U2.VOUT_SEL
- new net N$84: L9.2, U3.L
- new net N$85: C102.2, L8.1, U2.SW, U2.SW_2
- new net N$86: C106.1, U3.FC
- new net N$87: C102.1, U2.CBOOT
- new net N$88: R99.1, U3.PG
- new net N$89: IC9.SW, L10.2
- new net N$90: C108.1, IC13.BYPASS
- new net SWITCHED_IGN: C99.1, D6.A, D8.2
- net +3V3: now also C105.1, L9.1, U3.FB
- net EXT_PWR: now also D9.A
- net GND: now also C100.2, C101.2, C103.2, C104.2, C105.2, C106.2, C107.2, C108.2, C109.2, C110.2, D8.1, IC13.GND, IC9.EP, IC9.GND, IC9.MODE, R100.1, R101.1, R97.1, U2.AGND, U2.PAD, U2.PGND, U2.PGND_2, U2.SYNC_MODE, U3.GND, U3.PGND, U3.SYNC
- net HOST_RESET: now also R99.2
- net VDD: now also C104.1, IC9.FB, L10.1
Other:
- note added: "Connection of JTAG should also enable the board"
- moved on the sheet: C83, C84, C85, C86, C87, C88, C89, D4, D5, D7, IC13, IC9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

Commit message: Switch 3V3 LDO to fix compatibility with EN pins
Parts:
- removed C108: 0.01uF, rcl:C-USC0603
- removed IC13: TPS79133MDBVTEP, samacsys:TPS79133MDBVTEP
- removed R100, R101: 1k, rcl:R-US_R0603
- added IC17: LP5907QMFX-3.3Q1, samacsys:LP5907QMFX-3.3Q1
Connections:
- net N$88 renamed 3V3_SUPPLY_PGOOD
- removed net 1V2_SUPPLY_EN: IC9.EN, R100.2
- removed net 3V3_AD_SUPPLY_EN: IC13.!EN, R101.2
- removed net MAIN_SUPPLY_PGOOD: R98.1, U2.RESET_N, U3.EN
- removed net N$90: C108.1, IC13.BYPASS
- new net 5V_SUPPLY_PGOOD: IC17.EN, IC9.EN, R98.1, U2.RESET_N, U3.EN
- net +5V: now also IC17.IN; no longer IC13.IN
- net 3V3_AD_REF: now also IC17.OUT; no longer IC13.OUT
- net GND: now also IC17.GND; no longer C108.2, IC13.GND, R100.1, R101.1
Other:
- moved on the sheet: R99

Commit message: Add high side drivers
Parts:
- added C108, C111, C114, C116, C118, C120, C122, C124, C126, C128, C130, C132, C134, C136, C138, C140, C142, C144: 0.01uF, rcl:C-USC0603
- added C112, C113, C115, C117, C119, C121, C123, C125, C127, C129, C131, C133, C135, C137, C139, C141, C143, C145: 150nF, rcl:C-USC0603
- added D10, D11, D12, D13, D14, D15, D16, D17, D18, D19, D20, D21, D22, D23, D24, D25, D26, D27: BAT54SWFILMY, samacsys:BAT54SWFILMY
- added LED10, LED11, LED12, LED8: (no value), led:LEDCHIPLED_0603
- added R100, R101, R103, R104: 10k, rcl:R-US_R0603
- added R105, R106, R115, R120, R125, R130, R135, R140, R145, R150, R155, R160, R165, R170, R175, R180, R185, R190: 4, rcl:R-US_R1206
- added R107, R110, R111, R114, R116, R119, R121, R124, R126, R129, R131, R134, R136, R139, R141, R144, R146, R149, R151, R154, R156, R159, R161, R164, R166, R169, R171, R174, R176, R179, R181, R184, R186, R189, R191, R194: 4.7k, rcl:R-US_R0603
- added R108, R112, R117, R122, R127, R132, R137, R142, R147, R152, R157, R162, R167, R172, R177, R182, R187, R192: 2.74k, rcl:R-US_R0603
- added R109, R113, R118, R123, R128, R133, R138, R143, R148, R153, R158, R163, R168, R173, R178, R183, R188, R193: 1k, rcl:R-US_R0603
- added U?10, U?11, U?12, U?13, U?14, U?15, U?16, U?17, U?18, U?2, U?3, U?4, U?5, U?6, U?7, U?8, U?9: (no value), BTS50015-1TAD:BTS50015-1TAD
Connections:
- new net HIGHSIDE_0_EN: R154.2
- new net HIGHSIDE_0_OUTPUT: U?10.OUT1, U?10.OUT2, U?10.OUT3
- new net HIGHSIDE_10_EN: R114.2
- new net HIGHSIDE_10_OUTPUT: U?2.OUT1, U?2.OUT2, U?2.OUT3
- new net HIGHSIDE_11_EN: R119.2
- new net HIGHSIDE_11_OUTPUT: U?3.OUT1, U?3.OUT2, U?3.OUT3
- new net HIGHSIDE_12_EN: R124.2
- new net HIGHSIDE_12_OUTPUT: U?4.OUT1, U?4.OUT2, U?4.OUT3
- new net HIGHSIDE_13_EN: R129.2
- new net HIGHSIDE_13_OUTPUT: U?5.OUT1, U?5.OUT2, U?5.OUT3
- new net HIGHSIDE_14_EN: R134.2
- new net HIGHSIDE_14_OUTPUT: U?6.OUT1, U?6.OUT2, U?6.OUT3
- new net HIGHSIDE_15_EN: R139.2
- new net HIGHSIDE_15_OUTPUT: U?7.OUT1, U?7.OUT2, U?7.OUT3
- new net HIGHSIDE_16_EN: R144.2
- new net HIGHSIDE_16_OUTPUT: U?8.OUT1, U?8.OUT2, U?8.OUT3
- new net HIGHSIDE_17_EN: R149.2
- new net HIGHSIDE_17_OUTPUT: U?9.OUT1, U?9.OUT2, U?9.OUT3
- new net HIGHSIDE_1_EN: R159.2
- new net HIGHSIDE_1_OUTPUT: U?11.OUT1, U?11.OUT2, U?11.OUT3
- new net HIGHSIDE_2_EN: R164.2
- new net HIGHSIDE_2_OUTPUT: U?12.OUT1, U?12.OUT2, U?12.OUT3
- new net HIGHSIDE_3_EN: R169.2
- new net HIGHSIDE_3_OUTPUT: U?13.OUT1, U?13.OUT2, U?13.OUT3
- new net HIGHSIDE_4_EN: R174.2
- new net HIGHSIDE_4_OUTPUT: U?14.OUT1, U?14.OUT2, U?14.OUT3
- new net HIGHSIDE_5_EN: R179.2
- new net HIGHSIDE_5_OUTPUT: U?15.OUT1, U?15.OUT2, U?15.OUT3
- new net HIGHSIDE_6_EN: R184.2
- new net HIGHSIDE_6_OUTPUT: U?16.OUT1, U?16.OUT2, U?16.OUT3
- new net HIGHSIDE_7_EN: R189.2
- new net HIGHSIDE_7_OUTPUT: U?17.OUT1, U?17.OUT2, U?17.OUT3
- new net HIGHSIDE_8_EN: R194.2
- new net HIGHSIDE_8_OUTPUT: U?18.OUT1, U?18.OUT2, U?18.OUT3
- new net HIGHSIDE_9_EN: R110.2
- new net HIGHSIDE_9_OUTPUT: U?1.OUT1, U?1.OUT2, U?1.OUT3
- new net N$100: R115.1, U?3.GND
- new net N$101: R116.1, R117.1, U?3.IS
- new net N$102: C115.1, R118.1, R119.1, U?3.IN
- new net N$103: R120.1, U?4.GND
- new net N$104: R121.1, R122.1, U?4.IS
- new net N$105: C117.1, R123.1, R124.1, U?4.IN
- new net N$106: R125.1, U?5.GND
- new net N$107: R126.1, R127.1, U?5.IS
- new net N$108: C119.1, R128.1, R129.1, U?5.IN
- new net N$109: R130.1, U?6.GND
- new net N$110: R131.1, R132.1, U?6.IS
- new net N$111: C121.1, R133.1, R134.1, U?6.IN
- new net N$112: R135.1, U?7.GND
- new net N$113: R136.1, R137.1, U?7.IS
- new net N$114: C123.1, R138.1, R139.1, U?7.IN
- new net N$115: R140.1, U?8.GND
- new net N$116: R141.1, R142.1, U?8.IS
- new net N$117: C125.1, R143.1, R144.1, U?8.IN
- new net N$118: R145.1, U?9.GND
- new net N$119: R146.1, R147.1, U?9.IS
- new net N$120: C127.1, R148.1, R149.1, U?9.IN
- new net N$121: R150.1, U?10.GND
- new net N$122: R151.1, R152.1, U?10.IS
- new net N$123: C129.1, R153.1, R154.1, U?10.IN
- new net N$124: R155.1, U?11.GND
- new net N$125: R156.1, R157.1, U?11.IS
- new net N$126: C131.1, R158.1, R159.1, U?11.IN
- new net N$127: R160.1, U?12.GND
- new net N$128: R161.1, R162.1, U?12.IS
- new net N$129: C133.1, R163.1, R164.1, U?12.IN
- new net N$130: R165.1, U?13.GND
- new net N$131: R166.1, R167.1, U?13.IS
- new net N$132: C135.1, R168.1, R169.1, U?13.IN
- new net N$133: R170.1, U?14.GND
- new net N$134: R171.1, R172.1, U?14.IS
- new net N$135: C137.1, R173.1, R174.1, U?14.IN
- new net N$136: R175.1, U?15.GND
- new net N$137: R176.1, R177.1, U?15.IS
- new net N$138: C139.1, R178.1, R179.1, U?15.IN
- new net N$139: R180.1, U?16.GND
- new net N$140: R181.1, R182.1, U?16.IS
- new net N$141: C141.1, R183.1, R184.1, U?16.IN
- new net N$142: R185.1, U?17.GND
- new net N$143: R186.1, R187.1, U?17.IS
- new net N$144: C143.1, R188.1, R189.1, U?17.IN
- new net N$145: R190.1, U?18.GND
- new net N$146: R191.1, R192.1, U?18.IS
- new net N$147: C145.1, R193.1, R194.1, U?18.IN
- new net N$88: LED8.A, R100.2
- new net N$90: LED10.A, R101.2
- new net N$91: LED11.A, R103.2
- new net N$93: LED12.A, R104.2
- new net N$94: R106.1, U?1.GND
- new net N$95: R107.1, R108.1, U?1.IS
- new net N$96: R105.1, U?2.GND
- new net N$97: C112.1, R109.1, R110.1, U?1.IN
- new net N$98: R111.1, R112.1, U?2.IS
- new net N$99: C113.1, R113.1, R114.1, U?2.IN
- net +3V3: now also D10.K, D11.K, D12.K, D13.K, D14.K, D15.K, D16.K, D17.K, D18.K, D19.K, D20.K, D21.K, D22.K, D23.K, D24.K, D25.K, D26.K, D27.K, R103.1
- net +5V: now also R104.1
- net 3V3_AD_REF: now also R100.1
- net ADC0_10: now also C140.1, D25.A,K, R181.2
- net ADC0_3: now also C128.1, D19.A,K, R151.2
- net ADC0_4: now also C130.1, D20.A,K, R156.2
- net ADC0_6: now also C132.1, D21.A,K, R161.2
- net ADC0_7: now also C134.1, D22.A,K, R166.2
- net ADC0_8: now also C136.1, D23.A,K, R171.2
- net ADC0_9: now also C138.1, D24.A,K, R176.2
- net ADC1_0: now also C142.1, D26.A,K, R186.2
- net ADC1_1: now also C144.1, D27.A,K, R191.2
- net ADC1_10: now also C124.1, D17.A,K, R141.2
- net ADC1_11: now also C126.1, D18.A,K, R146.2
- net ADC1_2: now also C111.1, D10.A,K, R107.2
- net ADC1_4: now also C108.1, D11.A,K, R111.2
- net ADC1_5: now also C114.1, D12.A,K, R116.2
- net ADC1_6: now also C116.1, D13.A,K, R121.2
- net ADC1_7: now also C118.1, D14.A,K, R126.2
- net ADC1_8: now also C120.1, D15.A,K, R131.2
- net ADC1_9: now also C122.1, D16.A,K, R136.2
- net GND: now also C108.2, C111.2, C112.2, C113.2, C114.2, C115.2, C116.2, C117.2, C118.2, C119.2, C120.2, C121.2, C122.2, C123.2, C124.2, C125.2, C126.2, C127.2, C128.2, C129.2, C130.2, C131.2, C132.2, C133.2, C134.2, C135.2, C136.2, C137.2, C138.2, C139.2, C140.2, C141.2, C142.2, C143.2, C144.2, C145.2, D10.A, D11.A, D12.A, D13.A, D14.A, D15.A, D16.A, D17.A, D18.A, D19.A, D20.A, D21.A, D22.A, D23.A, D24.A, D25.A, D26.A, D27.A, LED10.C, LED11.C, LED12.C, LED8.C, R105.2, R106.2, R108.2, R109.2, R112.2, R113.2, R115.2, R117.2, R118.2, R120.2, R122.2, R123.2, R125.2, R127.2, R128.2, R130.2, R132.2, R133.2, R135.2, R137.2, R138.2, R140.2, R142.2, R143.2, R145.2, R147.2, R148.2, R150.2, R152.2, R153.2, R155.2, R157.2, R158.2, R160.2, R162.2, R163.2, R165.2, R167.2, R168.2, R170.2, R172.2, R173.2, R175.2, R177.2, R178.2, R180.2, R182.2, R183.2, R185.2, R187.2, R188.2, R190.2, R192.2, R193.2
- net VBATT: now also U?1.VS, U?10.VS, U?11.VS, U?12.VS, U?13.VS, U?14.VS, U?15.VS, U?16.VS, U?17.VS, U?18.VS, U?2.VS, U?3.VS, U?4.VS, U?5.VS, U?6.VS, U?7.VS, U?8.VS, U?9.VS
- net VDD: now also R101.1
Other:
- note added: "10. High Side Drivers (1/2)"
- note added: "10. High-side drivers (1/2)"
- note added: "11. High Side Drivers (2/2)"
- note added: "11. High-side drivers (2/2)"
- note added: "12. CAN"
- note added: "13. Modem"
- note added: "14. Connectors"
- note added: "RC lowpass on IS results in ~3400Hz cutoff"
- note removed: "10. High Side Drivers"
- note removed: "10. High-side drivers"
- note removed: "11. CAN"
- note removed: "12. Modem"
- note removed: "13. Connectors"
